Commit message: Fanuc

File: urdf/Fanuc.urdf.xacro (robot description, xacro)
@@ -12,5 +12,5 @@
 	<collision>
 		<geometry>
-			<mesh filename = "package://fanuc_motoman/meshes/Part 1.STL" scale = "0.001 0.001 0.001" />
+			<mesh filename = "package://fanuc/meshes/Part 1.STL" scale = "0.001 0.001 0.001" />
 		</geometry>
 	<origin xyz = "0 0 0" rpy = "0 0 0"/><!-- Best value <origin xyz = "0.105 0.09 0" rpy = "0 0 0" />-->
@@ -18,5 +18,5 @@
 	<visual>
  		<geometry>
-			<mesh filename = "package://fanuc_motoman/meshes/Part 1.STL" scale = "0.001 0.001 0.001" />
+			<mesh filename = "package://fanuc/meshes/Part 1.STL" scale = "0.001 0.001 0.001" />
 		</geometry>
 	<origin xyz = "0 0 0" rpy = "0 0 0"/><!-- Best value <origin xyz = "0.105 0.09 0" rpy = "0 0 0" />-->
@@ -48,5 +48,5 @@
 	<collision>
 	<geometry>
-		<mesh filename="package://fanuc_motoman/meshes/Part 2.STL" scale="0.001 0.001 0.001"/>
+		<mesh filename="package://fanuc/meshes/Part 2.STL" scale="0.001 0.001 0.001"/>
 	</geometry>
 		<origin xyz="-0.125 -0.110 0" rpy ="0 0 0"/>
@@ -54,5 +54,5 @@
 	<visual>
 	<geometry>
-		<mesh filename="package://fanuc_motoman/meshes/Part 2.STL" scale="0.001 0.001 0.001"/>
+		<mesh filename="package://fanuc/meshes/Part 2.STL" scale="0.001 0.001 0.001"/>
 	</geometry>
 		<origin xyz="-0.125 -0.110 0" rpy="0 0 0"/>
@@ -80,5 +80,5 @@
 		<origin xyz="-0.075 -0.1 -0.07" rpy="0 0 0"/>
 		<geometry>
-			<mesh filename="package://fanuc_motoman/meshes/Part 3.STL" scale="0.001 0.001 0.001"/>
+			<mesh filename="package://fanuc/meshes/Part 3.STL" scale="0.001 0.001 0.001"/>
 		</geometry>
 	</collision>
@@ -86,5 +86,5 @@
 		<origin xyz="-0.075 -0.1 -0.07" rpy="0 0 0"/>
 		<geometry>
-			<mesh filename = "package://fanuc_motoman/meshes/Part 3.STL" scale="0.001 0.001 0.001"/>
+			<mesh filename = "package://fanuc/meshes/Part 3.STL" scale="0.001 0.001 0.001"/>
 		</geometry>
 	</visual>
@@ -111,5 +111,5 @@
 		<origin xyz="-0.078 -0.068 -0.06" rpy="0 0 0"/>
 		<geometry>
-			<mesh filename="package://fanuc_motoman/meshes/Part 4.STL" scale="0.001 0.001 0.001"/>
+			<mesh filename="package://fanuc/meshes/Part 4.STL" scale="0.001 0.001 0.001"/>
 		</geometry>
 	</collision>
@@ -117,5 +117,5 @@
 		<origin xyz="-0.078 -0.068 -0.06" rpy="0 0 0"/>
 		<geometry>
-			<mesh filename="package://fanuc_motoman/meshes/Part 4.STL" scale="0.001 0.001 0.001"/>
+			<mesh filename="package://fanuc/meshes/Part 4.STL" scale="0.001 0.001 0.001"/>
 		</geometry>
 	</visual>
@@ -141,5 +141,5 @@
 		<origin xyz ="-0.1 -0.05 -0.045" rpy = "0 0 0" />
 		<geometry>
-			<mesh filename="package://fanuc_motoman/meshes/Part 5.STL" scale="0.001 0.001 0.001"/>
+			<mesh filename="package://fanuc/meshes/Part 5.STL" scale="0.001 0.001 0.001"/>
 		</geometry>
 	</collision>
@@ -147,5 +147,5 @@
 		<origin xyz ="-0.1 -0.05 -0.045" rpy = "0 0 0" />
 		<geometry>
-			<mesh filename="package://fanuc_motoman/meshes/Part 5.STL" scale="0.001 0.001 0.001"/>
+			<mesh filename="package://fanuc/meshes/Part 5.STL" scale="0.001 0.001 0.001"/>
 		</geometry>
 	</visual>
@@ -173,5 +173,5 @@
 		<origin xyz="-0.045 -.035 0.050" rpy ="0 1.57 0"/>
 		<geometry>
-			<mesh filename="package://fanuc_motoman/meshes/Part 6.STL" scale="0.001 0.001 0.001"/>
+			<mesh filename="package://fanuc/meshes/Part 6.STL" scale="0.001 0.001 0.001"/>
 		</geometry>
 	</collision>
@@ -179,5 +179,5 @@
 		<origin xyz="-0.045 -.035 0.050" rpy ="0 1.57 0"/>
 		<geometry>
-			<mesh filename="package://fanuc_motoman/meshes/Part 6.STL" scale="0.001 0.001 0.001"/>
+			<mesh filename="package://fanuc/meshes/Part 6.STL" scale="0.001 0.001 0.001"/>
 		</geometry>
 	</visual>
@@ -205,5 +205,5 @@
 		<origin xyz="-0.065 -0.065 0" rpy ="-1.57 0 0"/>
 		<geometry>
-			<mesh filename="package://fanuc_motoman/meshes/Gripper_base.STL" scale="0.001 0.001 0.001"/>
+			<mesh filename="package://fanuc/meshes/Gripper_base.STL" scale="0.001 0.001 0.001"/>
 		</geometry>
 	</collision>
@@ -211,5 +211,5 @@
 		<origin xyz="-0.065 -0.065 0" rpy ="-1.57 0 0"/>
 		<geometry>
-			<mesh filename="package://fanuc_motoman/meshes/Gripper_base.STL" scale="0.001 0.001 0.001"/>
+			<mesh filename="package://fanuc/meshes/Gripper_base.STL" scale="0.001 0.001 0.001"/>
 		</geometry>
 	</visual>
@@ -237,5 +237,5 @@
 		<origin xyz="0.075 0.038 0.075" rpy ="-1.57 0 3.14"/>
 		<geometry>
-			<mesh filename="package://fanuc_motoman/meshes/Gripper_finger.STL" scale="0.001 0.001 0.001"/>
+			<mesh filename="package://fanuc/meshes/Gripper_finger.STL" scale="0.001 0.001 0.001"/>
 		</geometry>
 	</collision>
@@ -243,5 +243,5 @@
 		<origin xyz="0.075 0.038 0.075" rpy ="-1.57 0 3.14"/>
 		<geometry>
-			<mesh filename="package://fanuc_motoman/meshes/Gripper_finger.STL" scale="0.001 0.001 0.001"/>
+			<mesh filename="package://fanuc/meshes/Gripper_finger.STL" scale="0.001 0.001 0.001"/>
 		</geometry>
 	</visual>
@@ -267,5 +267,5 @@
 		<origin xyz="-0.075 -0.038 0.075" rpy ="-1.57 0 0"/>
 		<geometry>
-			<mesh filename="package://fanuc_motoman/meshes/Gripper_finger.STL" scale="0.001 0.001 0.001"/>
+			<mesh filename="package://fanuc/meshes/Gripper_finger.STL" scale="0.001 0.001 0.001"/>
 		</geometry>
 	</collision>
@@ -273,5 +273,5 @@
 		<origin xyz="-0.075 -0.038 0.075" rpy ="-1.57 0 0"/>
 		<geometry>
-			<mesh filename="package://fanuc_motoman/meshes/Gripper_finger.STL" scale="0.001 0.001 0.001"/>
+			<mesh filename="package://fanuc/meshes/Gripper_finger.STL" scale="0.001 0.001 0.001"/>
 		</geometry>
 	</visual>
@@ -296,5 +296,5 @@
 		<origin xyz="-0.075 -0.038 0.075" rpy ="-1.57 0 0"/>
 		<geometry>
-			<mesh filename="package://fanuc_motoman/meshes/Gripper_finger.STL" scale="0.001 0.001 0.001"/>
+			<mesh filename="package://fanuc/meshes/Gripper_finger.STL" scale="0.001 0.001 0.001"/>
 		</geometry>
 	</collision>
@@ -302,5 +302,5 @@
 		<origin xyz="-0.075 -0.038 0.075" rpy ="-1.57 0 0"/>
 		<geometry>
-			<mesh filename="package://fanuc_motoman/meshes/Gripper_finger.STL" scale="0.001 0.001 0.001"/>
+			<mesh filename="package://fanuc/meshes/Gripper_finger.STL" scale="0.001 0.001 0.001"/>
 		</geometry>
 	</visual>
